File: Devboard.kicad_sch (KiCad schematic)
At the start: 27 parts, among them J1 0-13 pin, J2 A0-A5, J3 Power, P1 USB_C_Plug_USB2.0, SW1 SW_Push, U1 ATmega328-P, U2 CH340G, U3 L7805, Y1 12MHz, Y2 16MHz

Commit message: Pcb
Parts:
- removed C10, C11, C4, C5: 100nF, Capacitor_THT:C_Disc_D5.0mm_W2.5mm_P5.00mm, symbol Device:C
- removed C16: 10uF, Capacitor_THT:CP_Radial_D5.0mm_P2.00mm, symbol Device:C_Polarized
- R2: value 5v -> 5k
Connections:
- net +5V: now also U1.21 (AREF)
